Commit message: urdf-workinprogress

File: turntable_description/urdf/turntable.urdf (robot description, URDF)
Before this commit: robot turntable, 3 links, 2 joints
Links:
- added link base_link_inertia, mass 1.5; collision cylinder length=0.094 radius=0.1400; visual mesh filename=package://turntable_description/meshes/collision/turntable_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
- added link object_frame
- added link turntable_base
- link base_link: mass 1.5 -> None; geometry 
Joints:
- removed joint base_fixed
- added joint base_joint: type fixed, parent world, child base_link, origin xyz=0 0 0 rpy=0 0 0
- added joint base_link-base_link_inertia: type fixed, parent base_link, child base_link_inertia, origin xyz=0 0 0 rpy=0 0 0
- added joint base_link-turntable_base_joint: type fixed, parent base_link, child turntable_base, origin xyz=0 0 0 rpy=0 0 0
- added joint object_mount: type fixed, parent disc_link, child object_frame, origin xyz=0 0 0 rpy=0 0 0
- joint disc_joint: parent base_link -> base_link_inertia

File: turntable_description/urdf/turntable.urdf.xacro (robot description, xacro)
@@ -6,5 +6,4 @@
   <xacro:arg name="prefix" default=""/>
   <xacro:arg name="parent" default="world"/>
-  <xacro:arg name="use_nominal_extrinsics" default="false"/>
   <!-- Description config files -->
   <xacro:arg name="joint_limit_params" default="$(find turntable_description)/config/turntable/joint_limits.yaml"/>
@@ -31,5 +30,4 @@
     prefix="$(arg prefix)"
     parent="$(arg parent)"
-    use_nominal_extrinsics="$(arg use_nominal_extrinsics)"
     kinematics_parameters_file="$(arg kinematics_params)"
     joint_limits_parameters_file="$(arg joint_limit_params)"

File: turntable_description/urdf/turntable_macro.xacro (robot description, xacro)
@@ -9,5 +9,4 @@
       prefix
       parent
-      use_nominal_extrinsics
       kinematics_parameters_file
       joint_limits_parameters_file
@@ -85,5 +84,7 @@
     </link>
     <!-- Object-Co-Ordinate Frame -->
-    <link name="$${prefix}object_frame"/>
+    <link name="${prefix}object_frame"/>
+    <!-- ROS-Industrial 'base' frame - turntable base coordinates -->
+    <link name="${prefix}turntable_base"/>
     <!-- FIXED JOINT TO WORLD -->
     <joint name="${prefix}base_joint" type="fixed">
@@ -91,4 +92,11 @@
       <child link="${prefix}base_link"/>
       <origin xyz="0 0 0" rpy="0 0 0" />
+    </joint>
+    <!-- Coordinate System Alignment Joint -->
+    <joint name="${prefix}base_link-base_link_inertia" type="fixed">
+      <parent link="${prefix}base_link"/>
+      <child link="${prefix}base_link_inertia"/>
+      <!-- Coordinate alignment - add rotation here if needed for REP-103 compliance -->
+      <origin xyz="0 0 0" rpy="0 0 0"/>
     </joint>
     <!-- REVOLUTE JOINT -->
@@ -104,4 +112,16 @@
         velocity="${joint_limits.disc_joint.max_velocity}"/>
     </joint>
+    <!-- Object Mounted on Turntable: Standard frame reference on top of the disc_link -->
+    <joint name="${prefix}object_mount" type="fixed">
+      <parent link="${prefix}disc_link"/>
+      <child link="${prefix}object_frame"/>
+      <origin xyz="0 0 0" rpy="0 0 0"/>
+    </joint>
+    <!-- ROS-Industrial Base Frame -->
+    <joint name="${prefix}base_link-turntable_base_joint" type="fixed">
+      <origin xyz="0 0 0" rpy="0 0 0"/>
+      <parent link="${prefix}base_link"/>
+      <child link="${prefix}turntable_base"/>
+    </joint>
     <!-- TRANSMISSION BLOCK -->
     <xacro:turntable_transmission

File: turntable_moveit_config/config/turntable.ros2_control.xacro (robot description, xacro)
@@ -2,5 +2,5 @@
 <robot xmlns:xacro="http://www.ros.org/wiki/xacro">
     <xacro:macro name="turntable_ros2_control" params="name initial_positions_file">
-        <xacro:property name="initial_positions" value="${xacro.load_yaml(initial_positions_file)['initial_positions']}"/>
+        <xacro:property name="initial_positions" value="${load_yaml(initial_positions_file)['initial_positions']}"/>
         <ros2_control name="${name}" type="system">
             <hardware>
