Commit message: changed initial positions keys

File: turntable_description/urdf/turntable.urdf.xacro (robot description, xacro)
@@ -18,5 +18,5 @@
   <xacro:arg name="initial_positions_file" default="$(find turntable_description)/config/turntable/initial_positions.yaml"/>
   <xacro:property name="initial_positions_file" value="$(arg initial_positions_file)"/>
-  <xacro:property name="initial_positions" value="${xacro.load_yaml(initial_positions_file)['initial_positions']}"/>
+  <xacro:property name="initial_positions" value="${xacro.load_yaml(initial_positions_file)}"/>
   <!-- ros2_control plugin -->
   <xacro:turntable_ros2_control

File: turntable_moveit_config/config/turntable.ros2_control.xacro (robot description, xacro)
@@ -2,5 +2,5 @@
 <robot xmlns:xacro="http://www.ros.org/wiki/xacro">
     <xacro:macro name="turntable_ros2_control" params="name initial_positions_file">
-        <xacro:property name="initial_positions" value="${xacro.load_yaml(initial_positions_file)['initial_positions']}"/>
+        <xacro:property name="initial_positions" value="${xacro.load_yaml(initial_positions_file)}"/>
         <ros2_control name="${name}" type="system">
             <hardware>
