Commit message: Made changes to accomodate for 'turntable_forward_position_controller'. Removed 'turntable_controllers.yaml' and added 'ros2_controllers.yaml' instead, standardizing the nomenclature.

File: turntable_description/urdf/inc/turntable_common.xacro (robot description, xacro)
@@ -28,5 +28,5 @@
     </xacro:unless>
   </xacro:macro>
-  <xacro:macro name="read_model_data" params="joint_limits_parameters_file kinematics_parameters_file physical_parameters_file visual_parameters_file turntable_controllers_parameters_file">
+  <xacro:macro name="read_model_data" params="joint_limits_parameters_file kinematics_parameters_file physical_parameters_file visual_parameters_file ros2_controllers_parameters_file">
     <!-- Read .yaml files from disk, load content into properties -->
     <xacro:property name="config_joint_limit_parameters" value="${xacro.load_yaml(joint_limits_parameters_file)}"/>
@@ -34,5 +34,5 @@
     <xacro:property name="config_physical_parameters" value="${xacro.load_yaml(physical_parameters_file)}"/>
     <xacro:property name="config_visual_parameters" value="${xacro.load_yaml(visual_parameters_file)}"/>
-    <xacro:property name="congfig_turntable_controllers_parameters" value="${xacro.load_yaml(turntable_controllers_parameters_file)}"/>
+    <xacro:property name="config_ros2_controllers_parameters" value="${xacro.load_yaml(ros2_controllers_parameters_file)}"/>
     <!-- Extract subsections from yaml dictionaries -->
     <xacro:property name="sec_limits" value="${config_joint_limit_parameters['joint_limits']}"/>

File: turntable_description/urdf/turntable.urdf.xacro (robot description, xacro)
@@ -11,5 +11,5 @@
   <xacro:arg name="physical_params" default="$(find turntable_description)/config/turntable/physical_parameters.yaml"/>
   <xacro:arg name="visual_params" default="$(find turntable_description)/config/turntable/visual_parameters.yaml"/>
-  <xacro:arg name="turntable_controllers_params" default="$(find turntable_description)/config/turntable/turntable_controllers.yaml"/>
+  <xacro:arg name="ros2_controllers_params" default="$(find turntable_description)/config/turntable/ros2_controllers.yaml"/>
   <xacro:arg name="transmission_hw_interface" default=""/>
   <!-- ros2_control simulation toggle -->
@@ -34,5 +34,5 @@
     physical_parameters_file="$(arg physical_params)"
     visual_parameters_file="$(arg visual_params)"
-    turntable_controllers_parameters_file="$(arg turntable_controllers_params)"
+    ros2_controllers_parameters_file="$(arg ros2_controllers_params)"
     transmission_hw_interface="$(arg transmission_hw_interface)"/>
 </robot>

File: turntable_description/urdf/turntable_macro.xacro (robot description, xacro)
@@ -12,5 +12,5 @@
       joint_limits_parameters_file
       physical_parameters_file
-      turntable_controllers_parameters_file
+      ros2_controllers_parameters_file
       visual_parameters_file
       transmission_hw_interface:=hardware_interface/PositionJointInterface">
@@ -21,5 +21,5 @@
       physical_parameters_file="${physical_parameters_file}"
       visual_parameters_file="${visual_parameters_file}"
-      turntable_controllers_parameters_file="${turntable_controllers_parameters_file}"/>
+      ros2_controllers_parameters_file="${ros2_controllers_parameters_file}"/>
     <!-- Define the turntable name -->
     <!-- BASE LINK -->

File: turntable_moveit_config/config/turntable.ros2_control.xacro (robot description, xacro)
@@ -2,5 +2,5 @@
 <robot xmlns:xacro="http://www.ros.org/wiki/xacro">
     <xacro:macro name="turntable_ros2_control" params="name initial_positions_file">
-        <xacro:property name="initial_positions" value="${load_yaml(initial_positions_file)['initial_positions']}"/>
+        <xacro:property name="initial_positions" value="${xacro.load_yaml(initial_positions_file)['initial_positions']}"/>
         <ros2_control name="${name}" type="system">
             <hardware>
